File: Hardware/Qwiic Distance Sensor - VL53L1X.brd (EAGLE design)
At the start: 25.4 x 25.4 mm, 47 parts, among them J3 PTH, U2 VL53L1X

Commit message: Fixing issues
Parts:
- U$15: device buzzard_labels (14):QWIIC_DISTANCE7 -> buzzard_labels (7):QWIIC_DISTANCE0
- U$16: device buzzard_labels (14):VL53L1X8 -> buzzard_labels (7):VL53L1X1
- U$19: device buzzard_labels (15):QWIIC_DISTANCE9 -> buzzard_labels (7):QWIIC_DISTANCE0
- U$20: device buzzard_labels (15):VL53L1X10 -> buzzard_labels (7):VL53L1X1
- moved U$16 2.29 mm to (16.6, 11.7)
- moved U$15 1.33 mm to (19.1, 13.5)
Other:
- board text added: "v10"
- board text removed: "v01"
